File: kicad/usbwledc.kicad_sch (KiCad schematic)
At the start: 26 parts, among them J1 5V PAD, J10 USB_C_Receptacle_USB2.0, J2 D1 PAD, J3 GND PAD, J4 5V PAD, J5 D2 PAD, J6 GND PAD, J7 Conn_01x04_Pin, SW1 FLASH_SW, U1 CH340N, U2 AMS1117-3.3, U3 ESP32-WROOM-32

Commit message: v1.1
Parts:
- removed J7: Conn_01x04_Pin, Connector_PinHeader_2.54mm:PinHeader_1x04_P2.54mm_Vertical, symbol Connector:Conn_01x04_Pin
- removed MK1: ICS-43434, Sensor_Audio:InvenSense_ICS-43434-6_3.5x2.65mm, symbol Sensor_Audio:ICS-43434
- added J7: Accessories, Connector_PinHeader_2.54mm:PinHeader_1x06_P2.54mm_Vertical, symbol Connector:Conn_01x06_Pin
- added MK1: GSA4737, microphone:Microphone-6pin, symbol microphone:GSA4737
- C1, C2, C4: footprint Capacitor_SMD:C_0805_2012Metric -> Capacitor_SMD:C_0603_1608Metric; MPN C49678 -> C14663
- C3, C7: value 22uF -> 10uF; MPN C45783 -> C15850
- C6: footprint Capacitor_SMD:C_0805_2012Metric -> Capacitor_SMD:C_0603_1608Metric; MPN C28323 -> C15849
- C8: value 330uF -> 100uF; footprint Capacitor_THT:CP_Radial_D8.0mm_P3.50mm -> Capacitor_SMD:CP_Elec_5x5.4; symbol Device:C -> Device:C_Polarized; MPN C3008476 -> C131115
- J1, J2, J3, J4, J5, J6: footprint ProjectLibrary:SolderWirePad_1x01_SMD_3x6mm -> Library:SolderWirePad_1x01_SMD_3x6mm
- R1: footprint Resistor_SMD:R_0805_2012Metric -> Resistor_SMD:R_0603_1608Metric; MPN C149504 -> C25803
- R2, R3: footprint Resistor_SMD:R_0805_2012Metric -> Resistor_SMD:R_0603_1608Metric; MPN C17414 -> C25804
- R4, R5: footprint Resistor_SMD:R_0805_2012Metric -> Resistor_SMD:R_0603_1608Metric; MPN C27834 -> C23186
- SW1: footprint Button_Switch_SMD:SW_Tactile_SPST_NO_Straight_CK_PTS636Sx25SMTRLFS -> Button_Switch_SMD:SW_Push_1P1T_XKB_TS-1187A; MPN C3726366 -> C318884
Connections:
- net I2S_WS is gone; now on net I2S_SD: U3.37 (IO23)
- net +3V3: now also J7.2 (Pin_2), MK1.6 (VDD)
- net +5V: now also C8.1; no longer C8.2
- net GND: now also C8.2, J10.S1 (SHIELD), J7.1 (Pin_1), MK1.1 (GND), MK1.3 (GND); no longer C8.1
- net I2S_SCK: now also U3.36 (IO22), MK1.4 (SCK); no longer U3.33 (IO21)
- net I2S_SD: now also MK1.5 (SD); no longer U3.36 (IO22)
- net IO16: now also J7.6 (Pin_6)
- net IO17: now also J7.5 (Pin_5)
- net STRIP_DATA_1: now also U3.8 (IO32); no longer U3.9 (IO33)
- net STRIP_DATA_2: now also U3.9 (IO33); no longer U3.8 (IO32)
- net IO18: now reaches U3.30 (IO18)
- net IO18: now also J7.4 (Pin_4)
- net IO19: now reaches U3.31 (IO19)
- net IO19: now also J7.3 (Pin_3)
- net RELAY: no longer names the net of U3.12 (IO27)
- no-connect marks 23 -> 24
